Commit message: passed ur5+hand test

File: dexco/urdf/dexco.urdf (robot description, URDF)
Before this commit: robot dexco, 10 links, 9 joints
Links:
- removed link base_link
- added link hand_base_link
- link LL0: mass 0.08 -> 0.03
- link LL2: mass 0.08 -> 0.03
- link LL3: mass 0.08 -> 0.03
- link RL0: mass 0.08 -> 0.03
- link RL2: mass 0.08 -> 0.03
- link RL3: mass 0.08 -> 0.03
Joints:
- joint base: parent base_link -> hand_base_link
