Commit message: added readme

File: dexco/urdf/cylinder.urdf (robot description, URDF)
Before this commit: robot cylinder, 1 links, 0 joints
Links:
- link cylinder_link: mass 1.0 -> 0.3; geometry collision cylinder length=0.1 radius=0.035; visual cylinder length=0.1 radius=0.035

File: dexco/urdf/dexco.urdf (robot description, URDF)
Before this commit: robot dexco, 10 links, 9 joints
Joints:
- joint RJ0: limit lower=0 upper=0.022 effort=200 velocity=1 -> lower=-1 upper=1 effort=200 velocity=1
